Commit message: Simplify lane perception: two-line split, colour debug image

File: src/urdf_representations/qcar2/urdf/QCar2.urdf (robot description, URDF)
Before this commit: robot qcar2, 15 links, 14 joints
Links:
- link base_link: geometry collision box size=.03 .15 .115; collision box size=.037 .15 .115
- link csi_front: mass None -> 0.01; geometry collision box size=0.02 0.02 0.02; visual box size=0.02 0.02 0.02
- link hub_frontLeft: geometry visual mesh filename=file:///home/hammad/rosbot_ws/install/qcar2/share/qcar2/mes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 scale=0.001 0.001 0.001
- link hub_frontRight: geometry visual mesh filename=file:///home/hammad/rosbot_ws/install/qcar2/share/qcar2/mes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 scale=0.001 0.001 0.001
- link lidar: geometry visual cylinder length=0.0194 radius=0.04; visual mesh filename=file:///home/hammad/rosbot_ws/install/qcar2/share/qcar2/mes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 scale=0.1 0.1 0.1
- link wheel_frontLeft: geometry collision cylinder length=0.025 radius=0.033; visual mesh filename=file:///home/hammad/rosbot_ws/install/qcar2/share/qcar2/mes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 scale=0.001 0.001 0.001
- link wheel_frontRight: geometry collision cylinder length=0.025 radius=0.033; visual mesh filename=file:///home/hammad/rosbot_ws/install/qcar2/share/qcar2/mes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 scale=0.001 0.001 0.001
- link wheel_rearLeft: geometry collision cylinder length=0.025 radius=0.033; visual mesh filename=file:///home/hammad/rosbot_ws/install/qcar2/share/qcar2/mes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 scale=0.001 0.001 0.001
- link wheel_rearRight: geometry collision cylinder length=0.025 radius=0.033; visual mesh filename=file:///home/hammad/rosbot_ws/install/qcar2/share/qcar2/mes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 scale=0.001 0.001 0.001
Joints:
- joint csi_front_joint: origin xyz=0.198 0 0.1095 rpy=-1.5708 0 -1.5708 -> xyz=0.198 0 0.1095 rpy=0 0 0

Commit message: Working baseline: Simulation loads with fixed URDF paths

File: src/urdf_representations/qcar2/urdf/QCar2.urdf (robot description, URDF)
Before this commit: robot qcar2, 15 links, 14 joints
Links:
- link base_link: geometry collision box size=.03 .15 .115; collision box size=.037 .15 .115
- link hub_frontLeft: geometry visual mesh filename=file:///home/hajisaeed/qcar2_sim/install/qcar2/share/qcar2/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 scale=0.001 0.001 0.001
- link hub_frontRight: geometry visual mesh filename=file:///home/hajisaeed/qcar2_sim/install/qcar2/share/qcar2/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 scale=0.001 0.001 0.001
- link lidar: geometry visual cylinder length=0.0194 radius=0.04; visual mesh filename=file:///home/hajisaeed/qcar2_sim/install/qcar2/share/qcar2/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 scale=0.1 0.1 0.1
- link wheel_frontLeft: geometry collision cylinder length=0.025 radius=0.033; visual mesh filename=file:///home/hajisaeed/qcar2_sim/install/qcar2/share/qcar2/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 scale=0.001 0.001 0.001
- link wheel_frontRight: geometry collision cylinder length=0.025 radius=0.033; visual mesh filename=file:///home/hajisaeed/qcar2_sim/install/qcar2/share/qcar2/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 scale=0.001 0.001 0.001
- link wheel_rearLeft: geometry collision cylinder length=0.025 radius=0.033; visual mesh filename=file:///home/hajisaeed/qcar2_sim/install/qcar2/share/qcar2/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 scale=0.001 0.001 0.001
- link wheel_rearRight: geometry collision cylinder length=0.025 radius=0.033; visual mesh filename=file:///home/hajisaeed/qcar2_sim/install/qcar2/share/qcar2/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 scale=0.001 0.001 0.001
